File: hardware/Magnetic-Imaging-Tile.sch (EAGLE design)
At the start: 91 parts, among them U01 DRV5053, U02 DRV5053, U03 DRV5053, U04 DRV5053, U05 DRV5053, U06 DRV5053, U07 DRV5053, U08 CD74HC4067, U09 DRV5053, U10 DRV5053, U104 SN74HC509A, U105 SN74LVC1G139, U106 AD7680, U11 DRV5053, U12 DRV5053, U13 DRV5053, U14 DRV5053, U15 DRV5053, U16 DRV5053, U17 DRV5053, U18 CD74HC4067, U19 CD74HC4067, U20 DRV5053, U21 DRV5053, U22 DRV5053, U23 DRV5053, U24 DRV5053, U25 DRV5053, U26 DRV5053, U27 DRV5053, U28 CD74HC4067, U30 DRV5053, U31 DRV5053, U32 DRV5053, U33 DRV5053, U34 DRV5053, U35 DRV5053, U36 DRV5053, U37 DRV5053, U40 DRV5053, U41 DRV5053, U42 DRV5053, U43 DRV5053, U44 DRV5053, U45 DRV5053, U46 DRV5053, U47 DRV5053, U50 DRV5053, U51 DRV5053, U52 DRV5053, U53 DRV5053, U54 DRV5053, U55 DRV5053, U56 DRV5053, U57 DRV5053, U60 DRV5053, U61 DRV5053, U62 DRV5053, U63 DRV5053, U64 DRV5053, U65 DRV5053, U66 DRV5053, U67 DRV5053, U70 DRV5053, U71 DRV5053, U72 DRV5053, U73 DRV5053, U74 DRV5053, U75 DRV5053, U76 DRV5053, U77 DRV5053

Commit message: Update board with PROD_IDs
Parts:
- C1, C2, C3, C4, C5, C6, C7, C8: device SparkFun-Capacitors:4.7UF0603 -> SparkFun-Capacitors:4.7UF-0603-6.3V-(10%)
- U01, U02, U03, U04, U05, U06, U07, U09, U10, U11, U12, U13, U14, U15, U16, U17, U20, U21, U22, U23, U24, U25, U26, U27, U30, U31, U32, U33, U34, U35, U36, U37, U40, U41, U42, U43, U44, U45, U46, U47, U50, U51, U52, U53, U54, U55, U56, U57, U60, U61, U62, U63, U64, U65, U66, U67, U70, U71, U72, U73, U74, U75, U76, U77: device magneticimagertile:DRV5053 -> Magnetic-Imaging-Tile:DRV5053
- U104: value SN74HC509A -> SN74HC590A; device magneticimagertile:SN74HC509A -> Magnetic-Imaging-Tile:SN74HC590A
- U105: device magneticimagertile:SN74LVC1G139 -> Magnetic-Imaging-Tile:SN74LVC1G139
- U106: device magneticimagertile:AD7940 -> Magnetic-Imaging-Tile:AD7940
